File: ursus-flow.sch (EAGLE design)
At the start: 66 parts

Commit message: Update MT9V034 and MPU9250
Parts:
- removed C18, C5: 0.1uf, rcl:C-EUC0805
- removed R17, R9: 10k, resistor:R-EU_R0805W
Connections:
- removed net N$17: R9.1, U$4.BYPASS_CLKIN_N
- removed net N$18: R17.1, U$4.SER_DATAIN_N
- net +3V3: no longer C18.1, R17.2, R9.2
- net +5V: no longer C5.2
- net GND: no longer C18.2, C5.1, U$4.BYPASS_CLKIN_P, U$4.SER_DATAIN_P
Other:
- note added: "MT9V034(Breakboard Module)"
- note removed: "MT9V034(Module)"
Changed lines of the file:
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@@
 <part name="GND5" library="supply1" deviceset="GND" device=""/>
 <part name="P+5" library="supply1" deviceset="+5V" device=""/>
-<part name="C5" library="rcl" deviceset="C-EU" device="C0805" value="0.1uf"/>
-<part name="GND8" library="supply1" deviceset="GND" device=""/>
 <part name="C6" library="rcl" deviceset="C-EU" device="C0805" value="0.1uf"/>
 <part name="GND13" library="supply1" deviceset="GND" device=""/>
-<part name="C18" library="rcl" deviceset="C-EU" device="C0805" value="0.1uf"/>
-<part name="GND23" library="supply1" deviceset="GND" device=""/>
-<part name="GND29" library="supply1" deviceset="GND" device=""/>
-<part name="R9" library="resistor" deviceset="R-EU_" device="R0805W" value="10k"/>
-<part name="R17" library="resistor" deviceset="R-EU_" device="R0805W" value="10k"/>
-<part name="+3V9" library="supply1" deviceset="+3V3" device=""/>
 <part name="R18" library="resistor" deviceset="R-EU_" device="R0805W" value="1k"/>
 <part name="C19" library="rcl" deviceset="CPOL-US" device="B/3528-21W" value="100uf/10V"/>
@@
 <text x="-76.2" y="175.26" size="1.778" layer="98">Lidar</text>
 <text x="124.46" y="20.32" size="1.778" layer="98">MPU9250(Breakboard Module)</text>
-<text x="68.58" y="71.12" size="1.778" layer="98">MT9V034(Module)</text>
+<text x="68.58" y="71.12" size="1.778" layer="98">MT9V034(Breakboard Module)</text>
 <text x="10.16" y="213.36" size="1.778" layer="98">Power from UBEC (5V)</text>
 </plain>
@@
 <instance part="C13" gate="G$1" x="-55.88" y="114.3"/>
 <instance part="GND19" gate="1" x="-63.5" y="129.54" rot="R180"/>
-<instance part="+3V7" gate="G$1" x="177.8" y="12.7" rot="R270"/>
-<instance part="GND20" gate="1" x="170.18" y="5.08"/>
+<instance part="+3V7" gate="G$1" x="170.18" y="12.7" rot="R270"/>
+<instance part="GND20" gate="1" x="167.64" y="5.08"/>
 <instance part="SV3" gate="1" x="127" y="7.62"/>
 <instance part="R5" gate="G$1" x="-109.22" y="208.28"/>
@@
 <instance part="GND5" gate="1" x="2.54" y="81.28" rot="R90"/>
 <instance part="P+5" gate="1" x="40.64" y="66.04" rot="R90"/>
-<instance part="C5" gate="G$1" x="48.26" y="73.66"/>
-<instance part="GND8" gate="1" x="40.64" y="78.74" rot="R270"/>
 <instance part="C6" gate="G$1" x="17.78" y="10.16" rot="R270"/>
 <instance part="GND13" gate="1" x="7.62" y="10.16" rot="R270"/>
-<instance part="C18" gate="G$1" x="170.18" y="17.78" rot="R180"/>
-<instance part="GND23" gate="1" x="170.18" y="27.94" rot="R180"/>
-<instance part="GND29" gate="1" x="35.56" y="58.42" rot="R270"/>
-<instance part="R9" gate="G$1" x="152.4" y="58.42"/>
-<instance part="R17" gate="G$1" x="152.4" y="66.04"/>
-<instance part="+3V9" gate="G$1" x="167.64" y="63.5" rot="R270"/>
 <instance part="R18" gate="G$1" x="-139.7" y="53.34"/>
 <instance part="C19" gate="G$1" x="48.26" y="203.2"/>
@@
 </instance>
 <instance part="TEST_PAD2" gate="G$1" x="99.06" y="7.62" smashed="yes" rot="R90">
-<attribute name="NAME" x="109.22" y="4.445" size="1.778" layer="95" rot="R180"/>
+<attribute name="NAME" x="111.76" y="4.445" size="1.778" layer="95" rot="R180"/>
 <attribute name="TP_SIGNAL_NAME" x="100.33" y="10.16" size="1.778" layer="97" rot="R90"/>
 </instance>
@@
 <segment>
 <pinref part="SV3" gate="1" pin="5"/>
-<wire x1="134.62" y1="10.16" x2="170.18" y2="10.16" width="0.1524" layer="91"/>
+<wire x1="134.62" y1="10.16" x2="167.64" y2="10.16" width="0.1524" layer="91"/>
 <pinref part="GND20" gate="1" pin="GND"/>
-<wire x1="170.18" y1="10.16" x2="170.18" y2="7.62" width="0.1524" layer="91"/>
+<wire x1="167.64" y1="10.16" x2="167.64" y2="7.62" width="0.1524" layer="91"/>
 </segment>
 <segment>
@@
 </segment>
 <segment>
-<pinref part="GND8" gate="1" pin="GND"/>
-<pinref part="C5" gate="G$1" pin="1"/>
-<wire x1="43.18" y1="78.74" x2="48.26" y2="78.74" width="0.1524" layer="91"/>
-<wire x1="48.26" y1="78.74" x2="48.26" y2="76.2" width="0.1524" layer="91"/>
-</segment>
-<segment>
 <pinref part="GND13" gate="1" pin="GND"/>
 <pinref part="C6" gate="G$1" pin="2"/>
 <wire x1="10.16" y1="10.16" x2="12.7" y2="10.16" width="0.1524" layer="91"/>
-</segment>
-<segment>
-<pinref part="C18" gate="G$1" pin="2"/>
-<pinref part="GND23" gate="1" pin="GND"/>
-<wire x1="170.18" y1="22.86" x2="170.18" y2="25.4" width="0.1524" layer="91"/>
-</segment>
-<segment>
-<pinref part="GND29" gate="1" pin="GND"/>
-<pinref part="U$4" gate="G$1" pin="SER_DATAIN_P"/>
-<wire x1="38.1" y1="58.42" x2="58.42" y2="58.42" width="0.1524" layer="91"/>
-<wire x1="58.42" y1="58.42" x2="63.5" y2="58.42" width="0.1524" layer="91"/>
-<wire x1="58.42" y1="58.42" x2="58.42" y2="55.88" width="0.1524" layer="91"/>
-<pinref part="U$4" gate="G$1" pin="BYPASS_CLKIN_P"/>
-<wire x1="58.42" y1="55.88" x2="63.5" y2="55.88" width="0.1524" layer="91"/>
 </segment>
 <segment>
@@
 <pinref part="P+5" gate="1" pin="+5V"/>
 <pinref part="U$4" gate="G$1" pin="VCC"/>
-<wire x1="43.18" y1="66.04" x2="48.26" y2="66.04" width="0.1524" layer="91"/>
-<pinref part="C5" gate="G$1" pin="2"/>
-<wire x1="48.26" y1="66.04" x2="63.5" y2="66.04" width="0.1524" layer="91"/>
-<wire x1="48.26" y1="68.58" x2="48.26" y2="66.04" width="0.1524" layer="91"/>
+<wire x1="43.18" y1="66.04" x2="63.5" y2="66.04" width="0.1524" layer="91"/>
 </segment>
 </net>
@@
 <pinref part="SV3" gate="1" pin="6"/>
 <pinref part="+3V7" gate="G$1" pin="+3V3"/>
-<wire x1="134.62" y1="12.7" x2="170.18" y2="12.7" width="0.1524" layer="91"/>
-<pinref part="C18" gate="G$1" pin="1"/>
-<wire x1="170.18" y1="12.7" x2="175.26" y2="12.7" width="0.1524" layer="91"/>
-<wire x1="170.18" y1="15.24" x2="170.18" y2="12.7" width="0.1524" layer="91"/>
+<wire x1="134.62" y1="12.7" x2="167.64" y2="12.7" width="0.1524" layer="91"/>
 </segment>
 <segment>
@@
 <pinref part="R11" gate="G$1" pin="1"/>
 <wire x1="-147.32" y1="60.96" x2="-144.78" y2="60.96" width="0.1524" layer="91"/>
-</segment>
-<segment>
-<pinref part="R17" gate="G$1" pin="2"/>
-<wire x1="157.48" y1="66.04" x2="160.02" y2="66.04" width="0.1524" layer="91"/>
-<wire x1="160.02" y1="66.04" x2="160.02" y2="63.5" width="0.1524" layer="91"/>
-<pinref part="R9" gate="G$1" pin="2"/>
-<wire x1="160.02" y1="63.5" x2="160.02" y2="58.42" width="0.1524" layer="91"/>
-<wire x1="160.02" y1="58.42" x2="157.48" y2="58.42" width="0.1524" layer="91"/>
-<pinref part="+3V9" gate="G$1" pin="+3V3"/>
-<wire x1="165.1" y1="63.5" x2="160.02" y2="63.5" width="0.1524" layer="91"/>
 </segment>
 </net>
@@
 </segment>
 </net>
-<net name="N$17" class="0">
-<segment>
-<pinref part="U$4" gate="G$1" pin="BYPASS_CLKIN_N"/>
-<wire x1="121.92" y1="55.88" x2="144.78" y2="55.88" width="0.1524" layer="91"/>
-<wire x1="144.78" y1="55.88" x2="144.78" y2="58.42" width="0.1524" layer="91"/>
-<pinref part="R9" gate="G$1" pin="1"/>
-<wire x1="144.78" y1="58.42" x2="147.32" y2="58.42" width="0.1524" layer="91"/>
-</segment>
-</net>
-<net name="N$18" class="0">
-<segment>
-<pinref part="U$4" gate="G$1" pin="SER_DATAIN_N"/>
-<wire x1="121.92" y1="58.42" x2="142.24" y2="58.42" width="0.1524" layer="91"/>
-<wire x1="142.24" y1="58.42" x2="142.24" y2="66.04" width="0.1524" layer="91"/>
-<pinref part="R17" gate="G$1" pin="1"/>
-<wire x1="142.24" y1="66.04" x2="147.32" y2="66.04" width="0.1524" layer="91"/>
-</segment>
-</net>

Commit message: Arrange components
Parts:
- PWR_LED: value (none) -> PWR_LED
- SCHOTTKY1: value NSVR0320MW2T1G -> shottky1
- SCHOTTKY2: value NSVR0320MW2T1G -> shottky2
- renumbered P1 to [LIDAR], P2 to [SPI2], P3 to [UART2], P4 to [UART3], POWER_INDICATOR to PWR_LED, SV1 to [ST-LINK]
Changed lines of the file:
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@@
 <part name="LED2" library="led" deviceset="LED" device="SML0805"/>
 <part name="LED3" library="led" deviceset="LED" device="SML0805"/>
-<part name="POWER_INDICATOR" library="led" deviceset="LED" device="SML0805"/>
+<part name="PWR_LED" library="led" deviceset="LED" device="SML0805" value="PWR_LED"/>
 <part name="R1" library="resistor" deviceset="R-EU_" device="R0805W" value="220"/>
 <part name="R2" library="resistor" deviceset="R-EU_" device="R0805W" value="220"/>
@@
 <part name="+3V3" library="supply1" deviceset="+3V3" device=""/>
 <part name="+3V4" library="supply1" deviceset="+3V3" device=""/>
-<part name="SV1" library="con-lstb" deviceset="MA04-1" device=""/>
+<part name="[ST-LINK]" library="con-lstb" deviceset="MA04-1" device=""/>
 <part name="GND11" library="supply1" deviceset="GND" device=""/>
 <part name="U$3" library="usb_mirco_b" deviceset="MICRO-USB-RECEPTACLE" device="47589-0001"/>
@@
 <part name="U$4" library="MT9V034_MODULE" deviceset="MT9V034_MODULE" device=""/>
 <part name="GND27" library="supply1" deviceset="GND" device=""/>
-<part name="S1" library="switch-panasonic" deviceset="EVQPS" device="L/Q"/>
+<part name="S1" library="switch-panasonic" deviceset="EVQPS" device="L/Q" value=""/>
 <part name="GND28" library="supply1" deviceset="GND" device=""/>
 <part name="P+1" library="supply1" deviceset="+5V" device=""/>
@@
 <part name="C20" library="rcl" deviceset="CPOL-US" device="B/3528-21W" value="100uf/10V"/>
 <part name="GND30" library="supply1" deviceset="GND" device=""/>
-<part name="P1" library="jst-ph" deviceset="JST-PH4" device=""/>
-<part name="P2" library="jst-ph" deviceset="JST-PH6" device=""/>
-<part name="P3" library="jst-ph" deviceset="JST-PH4" device=""/>
-<part name="P4" library="jst-ph" deviceset="JST-PH4" device=""/>
-<part name="SCHOTTKY2" library="_mod_diode" deviceset="DIODE-" device="SOD323-W" value="NSVR0320MW2T1G"/>
-<part name="SCHOTTKY1" library="_mod_diode" deviceset="DIODE-" device="SOD323-W" value="NSVR0320MW2T1G"/>
+<part name="[LIDAR]" library="jst-ph" deviceset="JST-PH4" device=""/>
+<part name="[SPI2]" library="jst-ph" deviceset="JST-PH6" device=""/>
+<part name="[UART2]" library="jst-ph" deviceset="JST-PH4" device=""/>
+<part name="[UART3]" library="jst-ph" deviceset="JST-PH4" device=""/>
+<part name="SCHOTTKY2" library="_mod_diode" deviceset="DIODE-" device="SOD323-W" value="shottky2"/>
+<part name="SCHOTTKY1" library="_mod_diode" deviceset="DIODE-" device="SOD323-W" value="shottky1"/>
 <part name="TEST_PAD1" library="testpad" deviceset="TPSQ" device="TP20SQ"/>
 <part name="TEST_PAD2" library="testpad" deviceset="TPSQ" device="TP20SQ"/>
@@
 <instance part="LED2" gate="G$1" x="129.54" y="109.22" rot="R90"/>
 <instance part="LED3" gate="G$1" x="129.54" y="119.38" rot="R90"/>
-<instance part="POWER_INDICATOR" gate="G$1" x="81.28" y="208.28" rot="R90"/>
+<instance part="PWR_LED" gate="G$1" x="81.28" y="208.28" rot="R90"/>
 <instance part="R1" gate="G$1" x="142.24" y="99.06" rot="R180"/>
 <instance part="R2" gate="G$1" x="142.24" y="109.22" rot="R180"/>
@@
 <instance part="+3V3" gate="G$1" x="25.4" y="15.24"/>
 <instance part="+3V4" gate="G$1" x="-91.44" y="101.6" rot="R90"/>
-<instance part="SV1" gate="1" x="60.96" y="114.3"/>
+<instance part="[ST-LINK]" gate="1" x="60.96" y="114.3"/>
 <instance part="GND11" gate="1" x="71.12" y="101.6"/>
 <instance part="U$3" gate="G$1" x="17.78" y="167.64" rot="R180"/>
@@
 <instance part="C20" gate="G$1" x="114.3" y="170.18"/>
 <instance part="GND30" gate="1" x="48.26" y="193.04"/>
-<instance part="P1" gate="A" x="-73.66" y="165.1" rot="MR180"/>
-<instance part="P2" gate="A" x="-124.46" y="162.56" rot="MR180"/>
-<instance part="P3" gate="A" x="-73.66" y="203.2" rot="MR180"/>
-<instance part="P4" gate="A" x="-124.46" y="203.2" rot="MR180"/>
+<instance part="[LIDAR]" gate="A" x="-73.66" y="165.1" rot="MR180"/>
+<instance part="[SPI2]" gate="A" x="-124.46" y="162.56" rot="MR180"/>
+<instance part="[UART2]" gate="A" x="-73.66" y="203.2" rot="MR180"/>
+<instance part="[UART3]" gate="A" x="-124.46" y="203.2" rot="MR180"/>
 <instance part="SCHOTTKY2" gate="G$1" x="40.64" y="160.02" smashed="yes">
 <attribute name="NAME" x="33.02" y="152.8826" size="1.778" layer="95"/>
@@
 <net name="N$4" class="0">
 <segment>
-<pinref part="POWER_INDICATOR" gate="G$1" pin="C"/>
+<pinref part="PWR_LED" gate="G$1" pin="C"/>
 <pinref part="R4" gate="G$1" pin="2"/>
 <wire x1="86.36" y1="208.28" x2="93.98" y2="208.28" width="0.1524" layer="91"/>
@@
 </segment>
 <segment>
-<pinref part="SV1" gate="1" pin="1"/>
+<pinref part="[ST-LINK]" gate="1" pin="1"/>
 <pinref part="GND11" gate="1" pin="GND"/>
 <wire x1="68.58" y1="109.22" x2="71.12" y2="109.22" width="0.1524" layer="91"/>
@@
 <wire x1="-116.84" y1="200.66" x2="-111.76" y2="200.66" width="0.1524" layer="91"/>
 <wire x1="-111.76" y1="200.66" x2="-111.76" y2="198.12" width="0.1524" layer="91"/>
-<pinref part="P4" gate="A" pin="1"/>
+<pinref part="[UART3]" gate="A" pin="1"/>
 </segment>
 <segment>
@@
 <wire x1="-66.04" y1="200.66" x2="-60.96" y2="200.66" width="0.1524" layer="91"/>
 <wire x1="-60.96" y1="200.66" x2="-60.96" y2="198.12" width="0.1524" layer="91"/>
-<pinref part="P3" gate="A" pin="1"/>
+<pinref part="[UART2]" gate="A" pin="1"/>
 </segment>
 <segment>
@@
 <pinref part="GND16" gate="1" pin="GND"/>
 <wire x1="-104.14" y1="170.18" x2="-104.14" y2="175.26" width="0.1524" layer="91"/>
-<pinref part="P2" gate="A" pin="6"/>
+<pinref part="[SPI2]" gate="A" pin="6"/>
 </segment>
 <segment>
@@
 <wire x1="-66.04" y1="162.56" x2="-63.5" y2="162.56" width="0.1524" layer="91"/>
 <wire x1="-63.5" y1="162.56" x2="-63.5" y2="157.48" width="0.1524" layer="91"/>
-<pinref part="P1" gate="A" pin="1"/>
+<pinref part="[LIDAR]" gate="A" pin="1"/>
 </segment>
 <segment>
@@
 <wire x1="-35.56" y1="170.18" x2="-27.94" y2="170.18" width="0.1524" layer="91"/>
 <wire x1="-35.56" y1="167.64" x2="-35.56" y2="170.18" width="0.1524" layer="91"/>
-<pinref part="P1" gate="A" pin="4"/>
+<pinref part="[LIDAR]" gate="A" pin="4"/>
 </segment>
 <segment>
@@
 <segment>
 <pinref part="+3V2" gate="G$1" pin="+3V3"/>
-<pinref part="POWER_INDICATOR" gate="G$1" pin="A"/>
+<pinref part="PWR_LED" gate="G$1" pin="A"/>
 <wire x1="68.58" y1="208.28" x2="78.74" y2="208.28" width="0.1524" layer="91"/>
 </segment>
@@
 <pinref part="+3V5" gate="G$1" pin="+3V3"/>
 <wire x1="-116.84" y1="203.2" x2="-83.82" y2="203.2" width="0.1524" layer="91"/>
-<pinref part="P4" gate="A" pin="2"/>
+<pinref part="[UART3]" gate="A" pin="2"/>
 </segment>
 <segment>
 <pinref part="+3V6" gate="G$1" pin="+3V3"/>
 <wire x1="-116.84" y1="167.64" x2="-99.06" y2="167.64" width="0.1524" layer="91"/>
-<pinref part="P2" gate="A" pin="5"/>
+<pinref part="[SPI2]" gate="A" pin="5"/>
 </segment>
 <segment>
@@
 <wire x1="-33.02" y1="203.2" x2="-66.04" y2="203.2" width="0.1524" layer="91"/>
 <pinref part="+3V10" gate="G$1" pin="+3V3"/>
-<pinref part="P3" gate="A" pin="2"/>
+<pinref part="[UART2]" gate="A" pin="2"/>
 </segment>
 <segment>
@@
 <wire x1="-43.18" y1="167.64" x2="-66.04" y2="167.64" width="0.1524" layer="91"/>
 <label x="-63.5" y="167.64" size="1.778" layer="95"/>
-<pinref part="P1" gate="A" pin="3"/>
+<pinref part="[LIDAR]" gate="A" pin="3"/>
 </segment>
 </net>
@@
 <wire x1="-43.18" y1="165.1" x2="-66.04" y2="165.1" width="0.1524" layer="91"/>
 <label x="-63.5" y="165.1" size="1.778" layer="95"/>
-<pinref part="P1" gate="A" pin="2"/>
+<pinref part="[LIDAR]" gate="A" pin="2"/>
 </segment>
 </net>
@@
 <net name="STLINLK_SWDIO" class="0">
 <segment>
-<pinref part="SV1" gate="1" pin="3"/>
+<pinref part="[ST-LINK]" gate="1" pin="3"/>
 <wire x1="68.58" y1="114.3" x2="91.44" y2="114.3" width="0.1524" layer="91"/>
 <label x="71.12" y="114.3" size="1.778" layer="95"/>
@@
 <net name="STLINLK_SWCLK" class="0">
 <segment>
-<pinref part="SV1" gate="1" pin="2"/>
+<pinref part="[ST-LINK]" gate="1" pin="2"/>
 <wire x1="68.58" y1="111.76" x2="91.44" y2="111.76" width="0.1524" layer="91"/>
 <label x="71.12" y="111.76" size="1.778" layer="95"/>
@@
 <wire x1="-101.6" y1="160.02" x2="-116.84" y2="160.02" width="0.1524" layer="91"/>
 <label x="-114.3" y="160.02" size="1.778" layer="95"/>
-<pinref part="P2" gate="A" pin="2"/>
+<pinref part="[SPI2]" gate="A" pin="2"/>
 </segment>
 </net>
@@
 <wire x1="-101.6" y1="165.1" x2="-116.84" y2="165.1" width="0.1524" layer="91"/>
 <label x="-114.3" y="165.1" size="1.778" layer="95"/>
-<pinref part="P2" gate="A" pin="4"/>
+<pinref part="[SPI2]" gate="A" pin="4"/>
 </segment>
 </net>
@@
 <wire x1="-101.6" y1="162.56" x2="-116.84" y2="162.56" width="0.1524" layer="91"/>
 <label x="-114.3" y="162.56" size="1.778" layer="95"/>
-<pinref part="P2" gate="A" pin="3"/>
+<pinref part="[SPI2]" gate="A" pin="3"/>
 </segment>
 </net>
@@
 <wire x1="-104.14" y1="157.48" x2="-116.84" y2="157.48" width="0.1524" layer="91"/>
 <label x="-114.3" y="157.48" size="1.778" layer="95"/>
-<pinref part="P2" gate="A" pin="1"/>
+<pinref part="[SPI2]" gate="A" pin="1"/>
 </segment>
 </net>
@@
 <pinref part="R5" gate="G$1" pin="1"/>
 <wire x1="-116.84" y1="208.28" x2="-114.3" y2="208.28" width="0.1524" layer="91"/>
-<pinref part="P4" gate="A" pin="4"/>
+<pinref part="[UART3]" gate="A" pin="4"/>
 </segment>
 </net>
@@
 <pinref part="R6" gate="G$1" pin="1"/>
 <wire x1="-116.84" y1="205.74" x2="-114.3" y2="205.74" width="0.1524" layer="91"/>
-<pinref part="P4" gate="A" pin="3"/>
+<pinref part="[UART3]" gate="A" pin="3"/>
 </segment>
 </net>
@@
 <pinref part="R7" gate="G$1" pin="1"/>
 <wire x1="-66.04" y1="208.28" x2="-63.5" y2="208.28" width="0.1524" layer="91"/>
-<pinref part="P3" gate="A" pin="4"/>
+<pinref part="[UART2]" gate="A" pin="4"/>
 </segment>
 </net>
@@
 <pinref part="R8" gate="G$1" pin="1"/>
 <wire x1="-63.5" y1="205.74" x2="-66.04" y2="205.74" width="0.1524" layer="91"/>
-<pinref part="P3" gate="A" pin="3"/>
-</segment>
-</net>
+<pinref part="[UART2]" gate="A" pin="3"/>
+</segment>
+</net>
