File: ursus-flow.brd (EAGLE design)
At the start: 90.2 x 50.8 mm, 61 parts

Commit message: Keep routing
Parts:
- moved U$2 60.0 mm to (75.2, 48.8), turned to 270 degrees
- moved I2C3_SDA 56.5 mm to (72.6, 41.1), turned to 180 degrees
- moved I2C3_SCL 55.5 mm to (72.6, 43.7), turned to 180 degrees
- moved C6 47.7 mm to (68.8, 51.1), turned to 0 degrees
- moved R16 47.4 mm to (68.8, 46.2), turned to 180 degrees
- moved R11 47.3 mm to (68.8, 48.8), turned to 180 degrees
- moved [UART2] 11.4 mm to (50.8, 34.3)
- moved [UART3] 11.4 mm to (62.2, 34.3)
- moved R6 11.2 mm to (63.2, 38.4)
- moved R5 10.9 mm to (65.5, 38.4)
- moved R7 10.9 mm to (53.8, 38.4)
- moved R8 10.7 mm to (51.6, 38.4)
- moved C15 5.34 mm to (68.3, 62.5), turned to 270 degrees
- moved C11 0.76 mm to (52.8, 56.9)
- moved R13 0.51 mm to (89.2, 59.4), turned to 270 degrees
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Routing:
- net GND: track 241.3 -> 347.7 mm
- net +3V3: track 34.7 -> 133.8 mm, vias 0 -> 4
- net DCMI_D6: track 0.00 -> 54.4 mm, vias 0 -> 1
- net +5V: track 85.8 -> 138.8 mm, vias 2 -> 5
- net DCMI_D7: track 0.00 -> 46.6 mm, vias 0 -> 2
- net MPU9250_SPI1_CS: track 0.00 -> 43.4 mm, vias 0 -> 1
- net MPU9250_SPI1_SCK: track 0.00 -> 41.5 mm, vias 0 -> 1
- net MPU9250_SPI1_MOSI: track 0.00 -> 41.4 mm, vias 0 -> 1
- net MPU9250_SPI1_MISO: track 0.00 -> 40.8 mm
- net MT9V034_I2C1_SDA: track 0.00 -> 40.8 mm, vias 0 -> 1
- net MT9V034_I2C1_SCL: track 0.00 -> 34.9 mm, vias 0 -> 1
- net N$6: track 0.00 -> 27.3 mm
- net STLINLK_SWDIO: track 0.00 -> 27.1 mm, vias 0 -> 1
- net UART2_TX: track 0.00 -> 20.4 mm
- net AT24C08C_I2C3_SDA: track 9.93 -> 29.1 mm, vias 0 -> 3
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
Commit message: Layout is almost done
Routing:
- net +3V3: track 133.8 -> 194.8 mm, vias 4 -> 5
- net SPI2_MOSI: track 0.00 -> 46.5 mm, vias 0 -> 1
- net SPI2_MISO: track 0.00 -> 43.8 mm, vias 0 -> 1
- net GND: track 347.7 -> 391.4 mm, vias 1 -> 2
- net SPI2_CS: track 0.00 -> 39.6 mm, vias 0 -> 1
- net USB_OTG_FS_DM: track 0.00 -> 30.1 mm, vias 0 -> 2
- net USB_OTG_FS_DP: track 0.00 -> 27.4 mm, vias 0 -> 2
- net AT24C08C_A2: track 0.00 -> 22.2 mm, vias 0 -> 1
- net V_USB: track 3.03 -> 15.1 mm, vias 0 -> 2
- net +5V: track 138.8 -> 150.3 mm
- net DCMI_D6: track 54.4 -> 52.5 mm
- net DCMI_D7: track 46.6 -> 45.2 mm
- net MT9V034_I2C1_SCL: track 34.9 -> 36.1 mm
- net DCMI_D1: track 32.3 -> 31.7 mm
- net AT24C08C_I2C3_SDA: track 29.1 -> 28.5 mm

Commit message: Connect more traces
Routing:
- net SPI2_SCK: track 0.00 -> 21.8 mm, vias 0 -> 2
- net AT24C08C_I2C3_SCL: track 27.7 -> 37.7 mm
- net GND: track 391.4 -> 396.8 mm
- net N$4: track 0.00 -> 2.98 mm
- net +3V3: track 194.8 -> 195.5 mm
Changed lines of the file:
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@@
 <contactref element="PWR_LED" pad="C"/>
 <contactref element="R4" pad="2"/>
-<wire x1="35.3425" y1="76.2" x2="38.32" y2="76.2" width="0" layer="19" extent="1-1"/>
+<wire x1="35.3425" y1="76.2" x2="38.32" y2="76.2" width="0.4064" layer="1"/>
 </signal>
 <signal name="GND">
@@
 <wire x1="43.5" y1="54.61" x2="43.5" y2="53.274" width="0.3048" layer="1"/>
 <wire x1="43.5" y1="53.274" x2="43.942" y2="52.832" width="0.3048" layer="1"/>
+<wire x1="67.884" y1="51.054" x2="67.884" y2="50.988" width="0.3048" layer="16"/>
+<wire x1="67.884" y1="50.988" x2="69.088" y2="49.784" width="0.3048" layer="16"/>
+<wire x1="69.088" y1="49.784" x2="72.203" y2="49.784" width="0.3048" layer="16"/>
+<wire x1="72.203" y1="49.784" x2="72.584" y2="49.403" width="0.3048" layer="16"/>
 <wire x1="48.26" y1="66.99" x2="52.832" y2="68.3625" width="0" layer="19" extent="1-1"/>
 <wire x1="50.38" y1="63.63" x2="48.26" y2="66.99" width="0" layer="19" extent="1-1"/>
 <wire x1="46.736" y1="60.706" x2="50.38" y2="63.63" width="0" layer="19" extent="1-1"/>
 <wire x1="43.19" y1="57.79" x2="46.736" y2="57.634" width="0" layer="19" extent="1-1"/>
+<wire x1="42.23" y1="50.546" x2="42.164" y2="52.832" width="0" layer="19" extent="1-1"/>
 <wire x1="57.912" y1="53.086" x2="54.864" y2="52.324" width="0" layer="19" extent="1-16"/>
 <wire x1="61.976" y1="44.958" x2="60.706" y2="43.5" width="0" layer="19" extent="1-1"/>
-<wire x1="67.884" y1="51.054" x2="64.704" y2="46.228" width="0" layer="19" extent="1-16"/>
-<wire x1="72.584" y1="49.403" x2="67.884" y2="51.054" width="0" layer="19" extent="16-16"/>
+<wire x1="69.088" y1="49.784" x2="64.704" y2="46.228" width="0" layer="19" extent="1-16"/>
 <wire x1="16.155" y1="64.77" x2="16.51" y2="64.77" width="0" layer="19" extent="16-16"/>
 <wire x1="51.755" y1="74.47" x2="52.832" y2="68.3625" width="0" layer="19" extent="1-1"/>
-<wire x1="42.23" y1="50.546" x2="42.164" y2="52.832" width="0" layer="19" extent="1-1"/>
 </signal>
 <signal name="+5V">
@@
 <wire x1="61.23" y1="34.29" x2="61.23" y2="33.258" width="0.4064" layer="1"/>
 <wire x1="61.23" y1="33.258" x2="61.722" y2="32.766" width="0.4064" layer="1"/>
-<wire x1="61.722" y1="32.766" x2="68.326" y2="32.766" width="0.4064" layer="1"/>
-<wire x1="68.326" y1="32.766" x2="77.47" y2="32.766" width="0.4064" layer="1"/>
+<wire x1="61.722" y1="32.766" x2="68.072" y2="32.766" width="0.4064" layer="1"/>
+<wire x1="68.072" y1="32.766" x2="77.47" y2="32.766" width="0.4064" layer="1"/>
 <wire x1="77.47" y1="32.766" x2="77.978" y2="33.274" width="0.4064" layer="1"/>
 <wire x1="77.978" y1="33.274" x2="77.978" y2="34.242" width="0.4064" layer="1"/>
@@
 <wire x1="49.8" y1="36.052" x2="49.022" y2="36.83" width="0.4064" layer="1"/>
 <wire x1="49.022" y1="36.83" x2="43.434" y2="36.83" width="0.4064" layer="1"/>
-<wire x1="67.7815" y1="46.228" x2="67.7815" y2="39.4065" width="0.3048" layer="16"/>
-<wire x1="67.7815" y1="39.4065" x2="67.818" y2="39.37" width="0.3048" layer="16"/>
-<via x="67.818" y="39.37" extent="1-16" drill="0.6"/>
-<wire x1="67.818" y1="39.37" x2="67.818" y2="33.274" width="0.3048" layer="1"/>
-<wire x1="67.818" y1="33.274" x2="68.326" y2="32.766" width="0.3048" layer="1"/>
+<wire x1="67.7815" y1="46.228" x2="67.7815" y2="48.768" width="0.3048" layer="16"/>
+<wire x1="67.7815" y1="46.228" x2="67.7815" y2="43.9785" width="0.4064" layer="16"/>
+<wire x1="67.7815" y1="43.9785" x2="68.58" y2="43.18" width="0.4064" layer="16"/>
+<wire x1="68.58" y1="43.18" x2="68.58" y2="40.386" width="0.4064" layer="16"/>
+<wire x1="68.58" y1="40.386" x2="67.564" y2="39.37" width="0.4064" layer="16"/>
+<via x="67.564" y="39.37" extent="1-16" drill="0.6"/>
+<wire x1="67.564" y1="39.37" x2="67.564" y2="33.274" width="0.4064" layer="1"/>
+<wire x1="67.564" y1="33.274" x2="68.072" y2="32.766" width="0.4064" layer="1"/>
 <wire x1="79.2115" y1="58.42" x2="89.154" y2="60.4885" width="0" layer="19" extent="16-16"/>
 <wire x1="72.203" y1="51.054" x2="79.2115" y2="58.42" width="0" layer="19" extent="16-16"/>
@@
 <wire x1="49.88" y1="63.63" x2="50.038" y2="56.896" width="0" layer="19" extent="1-16"/>
 <wire x1="63.63" y1="61.88" x2="69.784" y2="51.054" width="0" layer="19" extent="1-16"/>
-<wire x1="67.7815" y1="46.228" x2="67.7815" y2="48.768" width="0.3048" layer="16"/>
 </signal>
 <signal name="USB_OTG_FS_DP">
@@
 <via x="69.85" y="57.658" extent="1-16" drill="0.6"/>
 <wire x1="69.8865" y1="48.768" x2="69.85" y2="48.768" width="0.3048" layer="16"/>
-<via x="68.834" y="52.578" extent="1-16" drill="0.6"/>
-<wire x1="68.834" y1="52.578" x2="68.834" y2="54.61" width="0.3048" layer="1"/>
-<via x="68.834" y="54.61" extent="1-16" drill="0.6"/>
-<wire x1="68.834" y1="54.61" x2="68.834" y2="57.404" width="0.3048" layer="16"/>
 <wire x1="69.85" y1="57.658" x2="69.088" y2="57.658" width="0.3048" layer="16"/>
 <wire x1="69.088" y1="57.658" x2="68.834" y2="57.404" width="0.3048" layer="16"/>
-<wire x1="68.834" y1="52.578" x2="68.834" y2="50.292" width="0.3048" layer="16"/>
-<wire x1="68.834" y1="50.292" x2="69.85" y2="49.276" width="0.3048" layer="16"/>
-<wire x1="69.85" y1="49.276" x2="69.85" y2="48.8045" width="0.3048" layer="16"/>
-<wire x1="69.85" y1="48.8045" x2="69.8865" y2="48.768" width="0.3048" layer="16"/>
+<via x="68.834" y="57.404" extent="1-16" drill="0.6"/>
+<wire x1="68.834" y1="57.404" x2="68.834" y2="49.911" width="0.3048" layer="1"/>
+<wire x1="68.834" y1="49.911" x2="70.612" y2="48.133" width="0.3048" layer="1"/>
+<wire x1="70.612" y1="48.133" x2="73.279" y2="48.133" width="0.3048" layer="1"/>
+<wire x1="73.279" y1="48.133" x2="74.422" y2="46.99" width="0.3048" layer="1"/>
+<wire x1="74.422" y1="46.99" x2="74.422" y2="46.228" width="0.3048" layer="1"/>
+<wire x1="74.422" y1="46.228" x2="74.168" y2="45.974" width="0.3048" layer="1"/>
+<wire x1="74.168" y1="45.974" x2="72.898" y2="45.974" width="0.3048" layer="1"/>
+<wire x1="72.898" y1="45.974" x2="72.644" y2="45.72" width="0.3048" layer="1"/>
+<via x="72.644" y="45.72" extent="1-16" drill="0.6"/>
+<wire x1="72.644" y1="45.72" x2="72.644" y2="43.688" width="0.3048" layer="16"/>
 </signal>
 <signal name="AT24C08C_I2C3_SDA">
@@
 <contactref element="U$1" pad="52"/>
 <contactref element="[SPI2]" pad="2"/>
-<wire x1="63.63" y1="50.38" x2="71.93" y2="34.29" width="0" layer="19" extent="1-1"/>
+<wire x1="71.93" y1="34.29" x2="71.93" y2="35.766" width="0.4064" layer="1"/>
+<wire x1="71.93" y1="35.766" x2="70.866" y2="36.83" width="0.4064" layer="1"/>
+<wire x1="63.63" y1="50.38" x2="64.682" y2="50.38" width="0.4064" layer="1"/>
+<wire x1="64.682" y1="50.38" x2="65.278" y2="49.784" width="0.4064" layer="1"/>
+<wire x1="65.278" y1="49.784" x2="66.04" y2="49.784" width="0.4064" layer="1"/>
+<wire x1="66.04" y1="49.784" x2="66.548" y2="49.276" width="0.4064" layer="1"/>
+<wire x1="66.548" y1="49.276" x2="66.548" y2="45.212" width="0.4064" layer="1"/>
+<via x="66.548" y="45.212" extent="1-16" drill="0.6"/>
+<wire x1="66.548" y1="45.212" x2="66.548" y2="41.91" width="0.4064" layer="16"/>
+<wire x1="66.548" y1="41.91" x2="67.564" y2="40.894" width="0.4064" layer="16"/>
+<via x="67.564" y="40.894" extent="1-16" drill="0.6"/>
+<wire x1="67.564" y1="40.894" x2="69.596" y2="40.894" width="0.4064" layer="1"/>
+<wire x1="69.596" y1="40.894" x2="70.866" y2="39.624" width="0.4064" layer="1"/>
+<wire x1="70.866" y1="39.624" x2="70.866" y2="36.83" width="0.4064" layer="1"/>
 </signal>
 <signal name="SPI2_MOSI">
