File: ursus-flow.brd (EAGLE design)
At the start: 90.2 x 50.8 mm, 61 parts

Commit message: Update component value
Parts:
- C20: value 100uf/10V -> 68uf/10V
- R1, R2: value 220 -> 1K
- R3: value 220 -> 10K
Changed lines of the file:
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@@
 <grid distance="0.1" unitdist="mm" unit="mm" style="lines" multiple="1" display="yes" altdistance="0.025" altunitdist="inch" altunit="inch"/>
 <layers>
-<layer number="1" name="Top" color="4" fill="1" visible="yes" active="yes"/>
+<layer number="1" name="Top" color="4" fill="1" visible="no" active="yes"/>
 <layer number="16" name="Bottom" color="1" fill="1" visible="yes" active="yes"/>
 <layer number="17" name="Pads" color="2" fill="1" visible="yes" active="yes"/>
@@
 <attribute name="VALUE" x="24.76" y="65.77" size="1.016" layer="28" rot="MR270"/>
 </element>
-<element name="C20" library="rcl" package="B/3528-21W" value="100uf/10V" x="17.78" y="64.77" smashed="yes" rot="MR180">
+<element name="C20" library="rcl" package="B/3528-21W" value="68uf/10V" x="17.78" y="64.77" smashed="yes" rot="MR180">
 <attribute name="NAME" x="16.1856" y="63.297" size="1.27" layer="26" rot="MR180"/>
 <attribute name="VALUE" x="14.56" y="67.695" size="1.27" layer="28" rot="MR180"/>
@@
 <attribute name="VALUE" x="35.33" y="76.74" size="1.27" layer="27" display="off"/>
 </element>
-<element name="R1" library="resistor" package="R0805W" value="220" x="74.93" y="71.12" smashed="yes" rot="R90">
+<element name="R1" library="resistor" package="R0805W" value="1K" x="74.93" y="71.12" smashed="yes" rot="R90">
 <attribute name="NAME" x="75.0062" y="67.8688" size="1.27" layer="25" rot="R90" align="center"/>
 <attribute name="VALUE" x="76.2" y="69.215" size="1.27" layer="27" rot="R90" align="center"/>
@@
 <attribute name="VALUE" x="46.101" y="72.136" size="1.27" layer="27" align="center"/>
 </element>
-<element name="R2" library="resistor" package="R0805W" value="220" x="72.39" y="71.12" smashed="yes" rot="R90">
+<element name="R2" library="resistor" package="R0805W" value="1K" x="72.39" y="71.12" smashed="yes" rot="R90">
 <attribute name="NAME" x="72.4154" y="67.8434" size="1.27" layer="25" rot="R90" align="center"/>
 <attribute name="VALUE" x="73.66" y="69.215" size="1.27" layer="27" rot="R90" align="center"/>
 </element>
-<element name="R3" library="resistor" package="R0805W" value="220" x="69.85" y="71.12" smashed="yes" rot="R90">
+<element name="R3" library="resistor" package="R0805W" value="10K" x="69.85" y="71.12" smashed="yes" rot="R90">
 <attribute name="NAME" x="69.8754" y="67.8434" size="1.27" layer="25" rot="R90" align="center"/>
 <attribute name="VALUE" x="71.12" y="69.215" size="1.27" layer="27" rot="R90" align="center"/>

Commit message: Update pull up resistors for mt9v034
Parts:
- R13: value 4.7k -> no need
- R15: value 4.7k -> 1k
Changed lines of the file:
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@@
 <attribute name="VALUE" x="41.656" y="38.989" size="1.27" layer="27" rot="R270" align="center"/>
 </element>
-<element name="R13" library="resistor" package="R0805W" value="4.7k" x="88.646" y="57.404" smashed="yes" rot="MR90">
+<element name="R13" library="resistor" package="R0805W" value="no need" x="88.646" y="57.404" smashed="yes" rot="MR90">
 <attribute name="NAME" x="89.8652" y="55.7276" size="1.27" layer="26" rot="MR90"/>
 <attribute name="VALUE" x="89.916" y="55.499" size="1.27" layer="28" rot="MR90"/>
@@
 <attribute name="VALUE" x="39.624" y="38.989" size="1.27" layer="27" rot="R270" align="center"/>
 </element>
-<element name="R15" library="resistor" package="R0805W" value="4.7k" x="80.264" y="58.42" smashed="yes" rot="MR180">
+<element name="R15" library="resistor" package="R0805W" value="1k" x="80.264" y="58.42" smashed="yes" rot="MR180">
 <attribute name="NAME" x="78.7654" y="60.8838" size="1.27" layer="26" rot="MR180"/>
 <attribute name="VALUE" x="78.359" y="60.96" size="1.27" layer="28" rot="MR180"/>
